File: door-ctrl/hardware-4/doorctrl-v4-gpio.sch (KiCad schematic (older format))
At the start: 33 parts, among them CON11 CONN_2_V, CON12 CONN_3_V, CON13 CONN_3_V, CON3 RJHSE-5085, CON4 RJHSE-5085, CON5 RJHSE-5085, K1 G5SB, K2 G5SB, Q3 BC817, Q4 BC817

Commit message: Starting out on the new firmware
Parts:
- CON11: symbol CONN_2_V -> borniers:CONN_2_V
- CON12, CON13: symbol CONN_3_V -> borniers:CONN_3_V
- CON3, CON4, CON5: symbol RJHSE-5085 -> amp-rj45-tap-up-with-leds:RJHSE-5085
- D10, D11: symbol DIODE-MINIMELF -> diode:DIODE-MINIMELF
- D4, D5: symbol LED -> doorctrl-v4-rescue:LED
- K1, K2: symbol G5SB -> g5sb:G5SB
- Q3, Q4: symbol BC817 -> bc817:BC817
- R10, R11, R12, R13, R16, R17, R18, R19, R22, R23, R24, R25, R33, R34, R35, R36, R37, R38, R39: symbol R -> doorctrl-v4-rescue:R
Connections:
- wire segments 103 -> 122
