File: door-ctrl/hardware-4/doorctrl-v4-net.sch (KiCad schematic (older format))
At the start: 38 parts, among them CON6 RJHSE-5085, U4 ENC28J60, U5 MC34063, X2 25MHz

Commit message: Starting out on the new firmware
Parts:
- C30, C31, C32, C33, C34, C35, C36, C39, C40, C41, C42, C43, C44: symbol C -> doorctrl-v4-rescue:C
- C37: symbol CAPAPOL -> doorctrl-v4-rescue:CAPAPOL
- CON6: symbol RJHSE-5085 -> amp-rj45-tap-up-with-leds:RJHSE-5085
- D8: symbol DIODESCH -> doorctrl-v4-rescue:DIODESCH
- L3, L4: symbol INDUCTOR -> doorctrl-v4-rescue:INDUCTOR
- R40, R41, R42, R43, R44, R45, R46, R47, R48, R49, R50, R51, R52, R53, R65, R67: symbol R -> doorctrl-v4-rescue:R
- TX1: symbol PE-68517L -> pulse-pe-68517-ethernet-trafo:PE-68517L
- U4: symbol ENC28J60 -> enc28j60:ENC28J60
- U5: symbol MC34063 -> doorctrl-v4-rescue:MC34063
- X2: symbol CRYSTAL -> doorctrl-v4-rescue:CRYSTAL
Connections:
- wire segments 111 -> 155
