File: door-ctrl/hardware-4/doorctrl-v4-psu.sch (KiCad schematic (older format))
At the start: 35 parts, among them U2 MC34063, U3 L4960

Commit message: Starting out on the new firmware
Parts:
- C10, C14, C15: symbol CAPAPOL -> doorctrl-v4-rescue:CAPAPOL
- C11, C12, C13, C16, C18, C19, C20, C22, C23, C24, C25, C45, C46, C9: symbol C -> doorctrl-v4-rescue:C
- D2, D3: symbol DIODESCH -> doorctrl-v4-rescue:DIODESCH
- H1, H2, H3, H4, H5: symbol MOUNTING -> mounting:MOUNTING
- L1, L2: symbol INDUCTOR -> doorctrl-v4-rescue:INDUCTOR
- R26, R27, R28, R29, R30, R31, R32: symbol R -> doorctrl-v4-rescue:R
- U2: symbol MC34063 -> doorctrl-v4-rescue:MC34063
- U3: symbol L4960 -> l4960:L4960
Connections:
- wire segments 47 -> 84
