File: door-ctrl/hardware-4/doorctrl-v4-rfid.sch (KiCad schematic (older format))
At the start: 19 parts, among them Q1 BC817, Q2 BC807, U1 LM358

Commit message: Starting out on the new firmware
Parts:
- C3, C4, C5, C6, C7, C8: symbol C -> doorctrl-v4-rescue:C
- D9: symbol DIODE-MINIMELF -> diode:DIODE-MINIMELF
- Q1: symbol BC817 -> bc817:BC817
- Q2: symbol BC807 -> bc807:BC807
- R1, R2, R3, R4, R5, R6, R7, R8, R9: symbol R -> doorctrl-v4-rescue:R
- U1: symbol LM358 -> linear:LM358
Connections:
- wire segments 43 -> 56
